File: eagle/nixie-tube-clock.brd (EAGLE design)
At the start: 156.4 x 70 mm, 93 parts, among them IC1 HV5622QC, IC2 HV5622QC, IC3 LM555D, IC4 MEGA8-AI, IC5 LD117ADT33TR, P1 1 k, Q1 7.3728 MHz, T1 BC547B, T2 TK3P50D, T3 BSS138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

Commit message: Beta version of PCB
Parts:
- moved - 109.6 mm to (116.8, 58.0)
- moved + 108.3 mm to (121.2, 58.0)
- moved T7 75.2 mm to (146.7, 42.6), turned to 270 degrees
- moved T8 73.7 mm to (9.97, 29.4), turned to 90 degrees
- moved C2 61.4 mm to (34.7, 31.5), turned to 90 degrees
- moved C3 59.3 mm to (21.6, 31.3), turned to 270 degrees
- moved T4 56.3 mm to (103.0, 29.6)
- moved T5 53.8 mm to (126.4, 43.1), turned to 270 degrees
- moved T9 52.0 mm to (78.8, 27.8)
- moved R2 51.2 mm to (41.4, 30.4)
- moved R4 51.0 mm to (21.7, 37.9), turned to 90 degrees
- moved R1 50.8 mm to (48.0, 35.9), turned to 90 degrees
- moved T1 49.3 mm to (32.4, 38.4), turned to 270 degrees
- moved T3 48.2 mm to (69.7, 28.6), turned to 90 degrees
- moved T2 48.0 mm to (11.9, 39.3), turned to 90 degrees
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Routing:
- net GND: track 0.00 -> 413.6 mm, vias 0 -> 12
- net +12V: track 147.5 -> 456.6 mm, vias 0 -> 5
- net +3V3: track 0.00 -> 117.9 mm, vias 0 -> 5
- net LED_D1: track 0.00 -> 92.2 mm, vias 0 -> 2
- net CLK: track 0.00 -> 82.7 mm, vias 0 -> 3
- net N$7: track 0.00 -> 78.3 mm, vias 0 -> 2
- net BL: track 0.00 -> 73.5 mm, vias 0 -> 2
- net LE: track 0.00 -> 72.2 mm, vias 0 -> 2
- net CASC: track 0.00 -> 69.9 mm, vias 0 -> 2
- net LED_D2: track 0.00 -> 66.4 mm, vias 0 -> 4
- net N$29: track 0.00 -> 58.9 mm, vias 0 -> 2
- net LED_B: track 194.8 -> 251.4 mm, vias 6 -> 7
- net V+: track 198.1 -> 252.5 mm, vias 0 -> 4
- net N$8: track 0.00 -> 48.4 mm, vias 0 -> 1
- net N$6: track 0.00 -> 40.8 mm, vias 0 -> 2
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Other:
- board size 156.4 x 70 mm -> 156.4 x 61.9 mm

Commit message: Pre-release version of PCB
Parts:
- added C10: 100 n, resistor:C1206
- moved R32 2.03 mm to (58.0, 21.1)
- moved GL4 0.76 mm to (106.1, 19.5)
- moved T2 0.53 mm to (12.1, 38.8)
- moved GL1 0.51 mm to (52.2, 16.1)
- moved T7 0.41 mm to (147.1, 42.6)
- moved GL2 0.25 mm to (106.1, 16.1)
- moved GL3 0.25 mm to (52.2, 19.4)
- moved T8 0.15 mm to (10.1, 29.4)
- moved R11 0.10 mm to (36.0, 16.4)
- moved T9 0.10 mm to (78.8, 27.9)
- moved IC5 0.05 mm to (138.7, 48.8)
Connections:
- net +3V3: now also C10.1
- net GND: now also C10.2
Routing:
- net GND: track 413.6 -> 386.2 mm, vias 12 -> 11
- net V+: track 252.5 -> 246.2 mm
- net +3V3: track 117.9 -> 122.7 mm
- net N$24: track 4.90 -> 7.19 mm
- net N$6: track 40.8 -> 42.8 mm
- net GLIMM_0: track 17.9 -> 18.8 mm
- net BL: track 73.5 -> 72.8 mm
